Commit message: Add new materials and apply them to kitchen and furniture models
- Introduced new materials for walls, windows, metal, and wood in furnitures.xacro.
- Updated visual elements in furnitures.xacro to use the new materials.
- Added new kitchen materials for white and gray finishes in kitchen.xacro.
- Applied new materials to various kitchen components, including cabinets, drawers, and countertops.

File: iai_apartment/urdf/furnitures.xacro (robot description, xacro)
@@ -1,3 +1,15 @@
 <robot xmlns:xacro="http://ros.org/wiki/xacro" name="furnitures">
+  <material name="apartment_wall_gray">
+    <color rgba="0.80 0.80 0.80 1"/>
+  </material>
+  <material name="apartment_window_blue">
+    <color rgba="0.16 0.22 0.28 1"/>
+  </material>
+  <material name="apartment_metal_gray">
+    <color rgba="0.68 0.68 0.68 1"/>
+  </material>
+  <material name="apartment_wood_brown">
+    <color rgba="0.55 0.45 0.32 1"/>
+  </material>
   <xacro:macro name="kitchen_macro" params="name parent *origin">
     <joint name="${name}" type="fixed">
@@ -18,4 +30,5 @@
           <mesh filename="package://iai_apartment/meshes/visual/walls.dae" />
         </geometry>
+        <material name="apartment_wall_gray"/>
       </visual>
       <!--collision>
@@ -35,4 +48,5 @@
           <mesh filename="package://iai_apartment/meshes/visual/windows.dae" />
         </geometry>
+        <material name="apartment_window_blue"/>
       </visual>
       <!--collision>
@@ -106,4 +120,5 @@
           <mesh filename="package://iai_apartment/meshes/visual/wardrobe.dae" />
         </geometry>
+        <material name="apartment_wall_gray"/>
       </visual>
       <collision>
@@ -210,4 +225,5 @@
           <mesh filename="package://iai_apartment/meshes/visual/wardrobe_door_left.dae" />
         </geometry>
+        <material name="apartment_metal_gray"/>
       </visual>
       <collision>
@@ -228,4 +244,5 @@
           <mesh filename="package://iai_apartment/meshes/visual/wardrobe_door_handle.dae" />
         </geometry>
+        <material name="apartment_metal_gray"/>
       </visual>
       <collision>
@@ -260,4 +277,5 @@
           <mesh filename="package://iai_apartment/meshes/visual/wardrobe_door_right.dae" />
         </geometry>
+        <material name="apartment_metal_gray"/>
       </visual>
       <collision>
@@ -278,4 +296,5 @@
           <mesh filename="package://iai_apartment/meshes/visual/wardrobe_door_handle.dae" />
         </geometry>
+        <material name="apartment_metal_gray"/>
       </visual>
       <collision>
@@ -308,4 +327,5 @@
           <mesh filename="package://iai_apartment/meshes/visual/armchair.dae" />
         </geometry>
+        <material name="apartment_metal_gray"/>
       </visual>
       <collision>
@@ -325,4 +345,5 @@
           <mesh filename="package://iai_apartment/meshes/visual/sofa.dae" />
         </geometry>
+        <material name="apartment_wall_gray"/>
       </visual>
       <collision>
@@ -342,4 +363,5 @@
           <mesh filename="package://iai_apartment/meshes/visual/coffee_table.dae" />
         </geometry>
+        <material name="apartment_wood_brown"/>
       </visual>
       <collision>
@@ -391,4 +413,5 @@
           <mesh filename="package://iai_apartment/meshes/visual/coffee_table_drawer.dae" />
         </geometry>
+        <material name="apartment_wood_brown"/>
       </visual>
       <collision>
@@ -433,4 +456,5 @@
           <mesh filename="package://iai_apartment/meshes/visual/bedside_table.dae" />
         </geometry>
+        <material name="apartment_wood_brown"/>
       </visual>
       <collision>

File: iai_apartment/urdf/kitchen.xacro (robot description, xacro)
@@ -1,3 +1,9 @@
 <robot xmlns:xacro="http://www.ros.org/wiki/xacro" name="kitchen">
+  <material name="apartment_kitchen_white">
+    <color rgba="0.08 0.08 0.09 1"/>
+  </material>
+  <material name="apartment_kitchen_gray">
+    <color rgba="0.12 0.12 0.14 1"/>
+  </material>
   <!-- Such is life in a kitchen : xacro -->
   <xacro:macro name="kitchen_macro" params="name parent *origin">
@@ -35,4 +41,5 @@
           <mesh filename="package://iai_apartment/meshes/cabinet01/IAICabinet1W60.dae" />
         </geometry>
+        <material name="apartment_kitchen_white"/>
       </visual>
       <collision>
@@ -56,4 +63,5 @@
           <mesh filename="package://iai_apartment/meshes/cabinet01/IAIDoorW60H80.dae" />
         </geometry>
+        <material name="apartment_kitchen_gray"/>
       </visual>
       <collision>
@@ -74,4 +82,5 @@
           <mesh filename="package://iai_apartment/meshes/handles/handle_horizontal.dae" />
         </geometry>
+        <material name="apartment_kitchen_gray"/>
       </visual>
       <collision>
@@ -96,5 +105,5 @@
           <mesh filename="package://iai_apartment/meshes/cabinet01/oven.dae" />
         </geometry>
-        <!-- <material name="oven_gray"/> -->
+        <material name="apartment_kitchen_gray"/>
       </visual>
       <collision>
@@ -117,4 +126,5 @@
           <mesh filename="package://iai_apartment/meshes/cabinet01/IAIDrawerW60H26.dae" />
         </geometry>
+        <material name="apartment_kitchen_gray"/>
       </visual>
       <collision>
@@ -135,4 +145,5 @@
           <mesh filename="package://iai_apartment/meshes/handles/handle_horizontal.dae" />
         </geometry>
+        <material name="apartment_kitchen_gray"/>
       </visual>
       <collision>
@@ -155,4 +166,5 @@
           <mesh filename="package://iai_apartment/meshes/cabinet01/IAIDrawerW60H53.dae" />
         </geometry>
+        <material name="apartment_kitchen_gray"/>
       </visual>
       <collision>
@@ -173,4 +185,5 @@
           <mesh filename="package://iai_apartment/meshes/handles/handle_horizontal.dae" />
         </geometry>
+        <material name="apartment_kitchen_gray"/>
       </visual>
       <collision>
@@ -233,4 +246,5 @@
           <mesh filename="package://iai_apartment/meshes/cabinet02/IAICabinet2W40H57.dae" />
         </geometry>
+        <material name="apartment_kitchen_gray"/>
       </visual>
       <collision>
@@ -261,4 +275,5 @@
           <mesh filename="package://iai_apartment/meshes/cabinet02/IAIDoorW40H212.dae" />
         </geometry>
+        <material name="apartment_kitchen_white"/>
       </visual>
       <collision>
@@ -279,4 +294,5 @@
           <mesh filename="package://iai_apartment/meshes/handles/handle_horizontal.dae" />
         </geometry>
+        <material name="apartment_kitchen_gray"/>
       </visual>
       <collision>
@@ -299,4 +315,5 @@
           <mesh filename="package://iai_apartment/meshes/cabinet02/IAIDrawerW40H10.dae" />
         </geometry>
+        <material name="apartment_kitchen_gray"/>
       </visual>
       <collision>
@@ -320,4 +337,5 @@
           <mesh filename="package://iai_apartment/meshes/cabinet02/IAIDrawerW40H22.dae" />
         </geometry>
+        <material name="apartment_kitchen_gray"/>
       </visual>
       <collision>
@@ -339,4 +357,5 @@
           <mesh filename="package://iai_apartment/meshes/cabinet03/IAICabinet3W60.dae" />
         </geometry>
+        <material name="apartment_kitchen_gray"/>
       </visual>
       <collision>
@@ -357,4 +376,5 @@
           <box size="0.036 0.56 1.2" />
         </geometry>
+        <material name="apartment_kitchen_white"/>
       </visual>
       <collision>
@@ -374,4 +394,5 @@
           <box size="0.036 0.5 1.2" />
         </geometry>
+        <material name="apartment_kitchen_white"/>
       </visual>
       <collision>
@@ -391,4 +412,5 @@
           <box size="0.036 0.5 1.2" />
         </geometry>
+        <material name="apartment_kitchen_white"/>
       </visual>
       <collision>
@@ -408,4 +430,5 @@
           <box size="0.5 0.535 0.036" />
         </geometry>
+        <material name="apartment_kitchen_white"/>
       </visual>
       <collision>
@@ -425,4 +448,5 @@
           <box size="0.5 0.535 0.036" />
         </geometry>
+        <material name="apartment_kitchen_white"/>
       </visual>
       <collision>
@@ -442,4 +466,5 @@
           <box size="0.5 0.535 0.036" />
         </geometry>
+        <material name="apartment_kitchen_white"/>
       </visual>
       <collision>
@@ -475,4 +500,5 @@
           <mesh filename="package://iai_apartment/meshes/cabinet03/IAIDoorW60H133.dae" />
         </geometry>
+        <material name="apartment_kitchen_gray"/>
       </visual>
       <collision>
@@ -493,4 +519,5 @@
           <mesh filename="package://iai_apartment/meshes/handles/handle_horizontal.dae" />
         </geometry>
+        <material name="apartment_kitchen_gray"/>
       </visual>
       <collision>
@@ -521,4 +548,5 @@
           <mesh filename="package://iai_apartment/meshes/cabinet03/IAIDoorW60H80.dae" />
         </geometry>
+        <material name="apartment_kitchen_gray"/>
       </visual>
       <collision>
@@ -539,4 +567,5 @@
           <mesh filename="package://iai_apartment/meshes/handles/handle_horizontal.dae" />
         </geometry>
+        <material name="apartment_kitchen_gray"/>
       </visual>
       <collision>
@@ -557,4 +586,5 @@
           <mesh filename="package://iai_apartment/meshes/cabinet04/IAIKitchenCabinet4W100.dae" />
         </geometry>
+        <material name="apartment_kitchen_white"/>
       </visual>
       <collision>
@@ -577,4 +607,5 @@
           <mesh filename="package://iai_apartment/meshes/cabinet04/IAIDoor1W100H40.dae" />
         </geometry>
+        <material name="apartment_kitchen_gray"/>
       </visual>
       <collision>
@@ -599,4 +630,5 @@
           <mesh filename="package://iai_apartment/meshes/cabinet04/IAIDoor2W100H40.dae" />
         </geometry>
+        <material name="apartment_kitchen_gray"/>
       </visual>
       <collision>
@@ -617,4 +649,5 @@
           <mesh filename="package://iai_apartment/meshes/handles/handle_horizontal.dae" />
         </geometry>
+        <material name="apartment_kitchen_gray"/>
       </visual>
       <collision>
@@ -635,4 +668,5 @@
           <mesh filename="package://iai_apartment/meshes/cabinet05/IAIKitchenCabinet5W60.dae" />
         </geometry>
+        <material name="apartment_kitchen_white"/>
       </visual>
       <collision>
@@ -655,4 +689,5 @@
           <mesh filename="package://iai_apartment/meshes/cabinet05/IAIKitchenDrawerW60H13.dae" />
         </geometry>
+        <material name="apartment_kitchen_gray"/>
       </visual>
       <collision>
@@ -673,4 +708,5 @@
           <mesh filename="package://iai_apartment/meshes/handles/handle_horizontal.dae" />
         </geometry>
+        <material name="apartment_kitchen_gray"/>
       </visual>
       <collision>
@@ -693,4 +729,5 @@
           <mesh filename="package://iai_apartment/meshes/cabinet05/IAIKitchenDrawerW60H26.dae" />
         </geometry>
+        <material name="apartment_kitchen_gray"/>
       </visual>
       <collision>
@@ -711,4 +748,5 @@
           <mesh filename="package://iai_apartment/meshes/handles/handle_horizontal.dae" />
         </geometry>
+        <material name="apartment_kitchen_gray"/>
       </visual>
       <collision>
@@ -731,4 +769,5 @@
           <mesh filename="package://iai_apartment/meshes/cabinet05/IAIKitchenDrawerW60H40.dae" />
         </geometry>
+        <material name="apartment_kitchen_gray"/>
       </visual>
       <collision>
@@ -749,4 +788,5 @@
           <mesh filename="package://iai_apartment/meshes/handles/handle_horizontal.dae" />
         </geometry>
+        <material name="apartment_kitchen_gray"/>
       </visual>
       <collision>
@@ -767,4 +807,5 @@
           <mesh filename="package://iai_apartment/meshes/cabinet06/IAIKitchenCabinet6W40.dae" />
         </geometry>
+        <material name="apartment_kitchen_white"/>
       </visual>
       <collision>
@@ -787,4 +828,5 @@
           <mesh filename="package://iai_apartment/meshes/cabinet06/IAIKitchenDrawerW40H13.dae" />
         </geometry>
+        <material name="apartment_kitchen_gray"/>
       </visual>
       <collision>
@@ -805,4 +847,5 @@
           <mesh filename="package://iai_apartment/meshes/handles/handle_horizontal.dae" />
         </geometry>
+        <material name="apartment_kitchen_gray"/>
       </visual>
       <collision>
@@ -825,4 +868,5 @@
           <mesh filename="package://iai_apartment/meshes/cabinet06/IAIKitchenDrawerW40H26.dae" />
         </geometry>
+        <material name="apartment_kitchen_gray"/>
       </visual>
       <collision>
@@ -843,4 +887,5 @@
           <mesh filename="package://iai_apartment/meshes/handles/handle_horizontal.dae" />
         </geometry>
+        <material name="apartment_kitchen_gray"/>
       </visual>
       <collision>
@@ -863,4 +908,5 @@
           <mesh filename="package://iai_apartment/meshes/cabinet06/IAIKitchenDrawerW40H40.dae" />
         </geometry>
+        <material name="apartment_kitchen_gray"/>
       </visual>
       <collision>
@@ -881,4 +927,5 @@
           <mesh filename="package://iai_apartment/meshes/handles/handle_horizontal.dae" />
         </geometry>
+        <material name="apartment_kitchen_gray"/>
       </visual>
       <collision>
@@ -899,4 +946,5 @@
           <mesh filename="package://iai_apartment/meshes/cabinet12/IAICabinet12W60.dae" />
         </geometry>
+        <material name="apartment_kitchen_white"/>
       </visual>
       <collision>
@@ -927,4 +975,5 @@
           <mesh filename="package://iai_apartment/meshes/cabinet12/IAIDoorW60H133.dae" />
         </geometry>
+        <material name="apartment_kitchen_gray"/>
       </visual>
       <collision>
@@ -956,4 +1005,5 @@
           <mesh filename="package://iai_apartment/meshes/cabinet12/IAIDoorW60H80.dae" />
         </geometry>
+        <material name="apartment_kitchen_gray"/>
       </visual>
       <collision>
@@ -976,4 +1026,5 @@
           <mesh filename="package://iai_apartment/meshes/cabinet07/IAIKitchenCabinet7W60.dae" />
         </geometry>
+        <material name="apartment_kitchen_gray"/>
       </visual>
       <collision>
@@ -996,4 +1047,5 @@
           <mesh filename="package://iai_apartment/meshes/cabinet07/IAIKitchenDoorW60H80.dae" />
         </geometry>
+        <material name="apartment_kitchen_gray"/>
       </visual>
       <collision>
@@ -1014,4 +1066,5 @@
           <mesh filename="package://iai_apartment/meshes/handles/handle_horizontal.dae" />
         </geometry>
+        <material name="apartment_kitchen_gray"/>
       </visual>
       <collision>
@@ -1035,4 +1088,5 @@
           <mesh filename="package://iai_apartment/meshes/cabinet07/dishwasher_drawer_middle.dae" />
         </geometry>
+        <material name="apartment_kitchen_gray"/>
       </visual>
       <collision>
@@ -1074,4 +1128,5 @@
           <mesh filename="package://iai_apartment/meshes/cabinet08/IAIKitchenCabinet8W60_v2.dae" />
         </geometry>
+        <material name="apartment_kitchen_gray"/>
       </visual>
       <collision>
@@ -1094,4 +1149,5 @@
           <mesh filename="package://iai_apartment/meshes/cabinet08/IAIKitchenDrawerW56H10.dae" />
         </geometry>
+        <material name="apartment_kitchen_gray"/>
       </visual>
       <collision>
@@ -1115,4 +1171,5 @@
           <mesh filename="package://iai_apartment/meshes/cabinet08/IAIKitchenDrawerW60H80.dae" />
         </geometry>
+        <material name="apartment_kitchen_white"/>
       </visual>
       <collision>
@@ -1133,4 +1190,5 @@
           <mesh filename="package://iai_apartment/meshes/handles/handle_horizontal.dae" />
         </geometry>
+        <material name="apartment_kitchen_gray"/>
       </visual>
       <collision>
@@ -1151,4 +1209,5 @@
           <mesh filename="package://iai_apartment/meshes/cabinet09/IAIKitchenCabinet9W60.dae" />
         </geometry>
+        <material name="apartment_kitchen_white"/>
       </visual>
       <collision>
@@ -1171,4 +1230,5 @@
           <mesh filename="package://iai_apartment/meshes/cabinet09/IAIKitchenDrawerW60H13.dae" />
         </geometry>
+        <material name="apartment_kitchen_gray"/>
       </visual>
       <collision>
@@ -1189,4 +1249,5 @@
           <mesh filename="package://iai_apartment/meshes/handles/handle_horizontal.dae" />
         </geometry>
+        <material name="apartment_kitchen_gray"/>
       </visual>
       <collision>
@@ -1209,4 +1270,5 @@
           <mesh filename="package://iai_apartment/meshes/cabinet09/IAIKitchenDrawerW60H26.dae" />
         </geometry>
+        <material name="apartment_kitchen_gray"/>
       </visual>
       <collision>
@@ -1227,4 +1289,5 @@
           <mesh filename="package://iai_apartment/meshes/handles/handle_horizontal.dae" />
         </geometry>
+        <material name="apartment_kitchen_gray"/>
       </visual>
       <collision>
@@ -1247,4 +1310,5 @@
           <mesh filename="package://iai_apartment/meshes/cabinet09/IAIKitchenDrawerW60H40.dae" />
         </geometry>
+        <material name="apartment_kitchen_gray"/>
       </visual>
       <collision>
@@ -1265,4 +1329,5 @@
           <mesh filename="package://iai_apartment/meshes/handles/handle_horizontal.dae" />
         </geometry>
+        <material name="apartment_kitchen_gray"/>
       </visual>
       <collision>
@@ -1283,4 +1348,5 @@
           <mesh filename="package://iai_apartment/meshes/cabinet10/IAIKitchenCabinet9W40.dae" />
         </geometry>
+        <material name="apartment_kitchen_white"/>
       </visual>
       <collision>
@@ -1303,4 +1369,5 @@
           <mesh filename="package://iai_apartment/meshes/cabinet10/IAIKitchenDrawerW40H13.dae" />
         </geometry>
+        <material name="apartment_kitchen_gray"/>
       </visual>
       <collision>
@@ -1321,4 +1388,5 @@
           <mesh filename="package://iai_apartment/meshes/handles/handle_horizontal.dae" />
         </geometry>
+        <material name="apartment_kitchen_gray"/>
       </visual>
       <collision>
@@ -1341,4 +1409,5 @@
           <mesh filename="package://iai_apartment/meshes/cabinet10/IAIKitchenDrawerW40H26.dae" />
         </geometry>
+        <material name="apartment_kitchen_gray"/>
       </visual>
       <collision>
@@ -1359,4 +1428,5 @@
           <mesh filename="package://iai_apartment/meshes/handles/handle_horizontal.dae" />
         </geometry>
+        <material name="apartment_kitchen_gray"/>
       </visual>
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